Commit message: dual robot settings

File: construct_description/urdf_0528/construct_robot_0528 copy.urdf (robot description, URDF)
Before this commit: robot construct_robot_0528, 56 links, 55 joints
Links:
- link base_link: geometry collision mesh filename=../meshes_0528/base_link_optimized.stl; visual mesh filename=../meshes_0528/base_link_optimized.stl
- link controlbox_link: geometry collision mesh filename=../meshes_0528/controlbox_link_optimized.stl; visual mesh filename=../meshes_0528/controlbox_link_optimized.stl
- link helios_link: geometry collision mesh filename=../meshes_0528/helios_link_optimized.stl; visual mesh filename=../meshes_0528/helios_link_optimized.stl
- link left_D435_link: geometry collision mesh filename=../meshes_0528/left_D435_link_optimized.stl; visual mesh filename=../meshes_0528/left_D435_link_optimized.stl
- link left_manipulator_base_link: geometry collision mesh filename=../meshes_0528/left_manipulator_base_link_optimized.stl; visual mesh filename=../meshes_0528/left_manipulator_base_link_optimized.stl
- link left_manipulator_link1: geometry collision mesh filename=../meshes_0528/left_manipulator_link1_optimized.stl; visual mesh filename=../meshes_0528/left_manipulator_link1_optimized.stl
- link left_manipulator_link2: geometry collision mesh filename=../meshes_0528/left_manipulator_link2_optimized.stl; visual mesh filename=../meshes_0528/left_manipulator_link2_optimized.stl
- link left_manipulator_link3: geometry collision mesh filename=../meshes_0528/left_manipulator_link3_optimized.stl; visual mesh filename=../meshes_0528/left_manipulator_link3_optimized.stl
- link left_manipulator_link4: geometry collision mesh filename=../meshes_0528/left_manipulator_link4_optimized.stl; visual mesh filename=../meshes_0528/left_manipulator_link4_optimized.stl
- link left_manipulator_link5: geometry collision mesh filename=../meshes_0528/left_manipulator_link5_optimized.stl; visual mesh filename=../meshes_0528/left_manipulator_link5_optimized.stl
- link left_manipulator_link6: geometry collision mesh filename=../meshes_0528/left_manipulator_link6_optimized.stl; visual mesh filename=../meshes_0528/left_manipulator_link6_optimized.stl
- link left_manipulator_link_ee: geometry collision mesh filename=../meshes_0528/left_manipulator_link_ee_optimized.stl; visual mesh filename=../meshes_0528/left_manipulator_link_ee_optimized.stl
- link right_D435_link: geometry collision mesh filename=../meshes_0528/right_D435_link_optimized.stl; visual mesh filename=../meshes_0528/right_D435_link_optimized.stl
- link right_manipulator_base_link: geometry collision mesh filename=../meshes_0528/right_manipulator_base_link_optimized.stl; visual mesh filename=../meshes_0528/right_manipulator_base_link_optimized.stl
- link right_manipulator_link1: geometry collision mesh filename=../meshes_0528/right_manipulator_link1_optimized.stl; visual mesh filename=../meshes_0528/right_manipulator_link1_optimized.stl
- link right_manipulator_link2: geometry collision mesh filename=../meshes_0528/right_manipulator_link2_optimized.stl; visual mesh filename=../meshes_0528/right_manipulator_link2_optimized.stl
- link right_manipulator_link3: geometry collision mesh filename=../meshes_0528/right_manipulator_link3_optimized.stl; visual mesh filename=../meshes_0528/right_manipulator_link3_optimized.stl
- link right_manipulator_link4: geometry collision mesh filename=../meshes_0528/right_manipulator_link4_optimized.stl; visual mesh filename=../meshes_0528/right_manipulator_link4_optimized.stl
- link right_manipulator_link5: geometry collision mesh filename=../meshes_0528/right_manipulator_link5_optimized.stl; visual mesh filename=../meshes_0528/right_manipulator_link5_optimized.stl
- link right_manipulator_link6: geometry collision mesh filename=../meshes_0528/right_manipulator_link6_optimized.stl; visual mesh filename=../meshes_0528/right_manipulator_link6_optimized.stl
- link right_manipulator_link_ee: geometry collision mesh filename=../meshes_0528/right_manipulator_link_ee_optimized.stl; visual mesh filename=../meshes_0528/right_manipulator_link_ee_optimized.stl
- link robot_base_link: geometry collision mesh filename=../meshes_0528/robot_base_link_optimized.stl; visual mesh filename=../meshes_0528/robot_base_link_optimized.stl
- link robot_head_base_link: geometry collision mesh filename=../meshes_0528/robot_head_base_link_optimized.stl; visual mesh filename=../meshes_0528/robot_head_base_link_optimized.stl
- link robot_head_rev_link1: geometry collision mesh filename=../meshes_0528/robot_head_rev_link1_optimized.stl; visual mesh filename=../meshes_0528/robot_head_rev_link1_optimized.stl
- link robot_head_rev_link2: geometry collision mesh filename=../meshes_0528/robot_head_rev_link2_optimized.stl; visual mesh filename=../meshes_0528/robot_head_rev_link2_optimized.stl
- link testbed_link: geometry collision mesh filename=../meshes_0528/testbed_link_optimized.stl; visual mesh filename=../meshes_0528/testbed_link_optimized.stl
- link zed2i_link: geometry collision mesh filename=../meshes_0528/zed2i_link_optimized.stl; visual mesh filename=../meshes_0528/zed2i_link_optimized.stl
- link zed_bracket_link: geometry collision mesh filename=../meshes_0528/zed_bracket_link_optimized.stl; visual mesh filename=../meshes_0528/zed_bracket_link_optimized.stl
Joints:
- joint left_manipulator_base_joint: origin xyz=0.25 0 1.0002 rpy=0 0 3.141592653589793 -> xyz=-0.25 0 1.0002 rpy=0 0 0
- joint right_manipulator_base_joint: origin xyz=-0.25 0 1.00019999999931 rpy=0 0 3.141592653589793 -> xyz=0.24999999999997 0 1.00019999999931 rpy=0 0 0

File: construct_description/urdf_0528/construct_robot_0528.control.urdf.xacro (robot description, xacro)
@@ -4,10 +4,6 @@
   <xacro:arg name="left_robot_ip" default="192.168.1.11" />
   <xacro:arg name="cb_simulation" default="false" />
-  <xacro:arg name="use_fake_left_hardware" default="true" />
-  <xacro:arg name="use_fake_right_hardware" default="true" />
-  <xacro:arg name="use_initial_left_positions" default="true" />
-  <xacro:arg name="use_initial_right_positions" default="true" />
-  <xacro:arg name="initial_positions_file"
-             default="$(find construct_description)/config/initial_positions.yaml" />
+  <xacro:arg name="use_fake_left_hardware" default="false" />
+  <xacro:arg name="use_fake_right_hardware" default="false" />
   <xacro:arg name="fake_sensor_commands" default="false" />
   <xacro:include filename="$(find construct_description)/urdf_0528/construct_robot_0528.urdf" />
@@ -19,7 +15,4 @@
       use_fake_left_hardware="$(arg use_fake_left_hardware)"
       use_fake_right_hardware="$(arg use_fake_right_hardware)"
-      use_initial_left_positions="$(arg use_initial_left_positions)"
-      use_initial_right_positions="$(arg use_initial_right_positions)"
-      initial_positions_file="$(arg initial_positions_file)"
       fake_sensor_commands="$(arg fake_sensor_commands)" />
 </robot>

File: construct_description/urdf_0528/construct_robot_0528.ros2_control.xacro (robot description, xacro)
@@ -3,7 +3,5 @@
   <xacro:macro
     name="construct_robot_0528_ros2_control"
-    params="left_robot_ip right_robot_ip cb_simulation:=false use_fake_left_hardware:=true use_fake_right_hardware:=false use_initial_left_positions:=true use_initial_right_positions:=true initial_positions_file fake_sensor_commands:=false">
-    <xacro:property name="initial_positions"
-                    value="${xacro.load_yaml(initial_positions_file)['initial_positions']}" />
+    params="left_robot_ip right_robot_ip cb_simulation:=false use_fake_left_hardware:=false use_fake_right_hardware:=false fake_sensor_commands:=false">
     <xacro:macro name="configure_rb_joint" params="joint_name initial_value:=0.0">
       <joint name="${joint_name}">
@@ -35,10 +33,10 @@
         </xacro:unless>
       </hardware>
-      <xacro:configure_rb_joint joint_name="left_manipulator_joint1" initial_value="${initial_positions['left_manipulator_joint1'] if use_initial_left_positions else 0.0}" />
-      <xacro:configure_rb_joint joint_name="left_manipulator_joint2" initial_value="${initial_positions['left_manipulator_joint2'] if use_initial_left_positions else 0.0}" />
-      <xacro:configure_rb_joint joint_name="left_manipulator_joint3" initial_value="${initial_positions['left_manipulator_joint3'] if use_initial_left_positions else 0.0}" />
-      <xacro:configure_rb_joint joint_name="left_manipulator_joint4" initial_value="${initial_positions['left_manipulator_joint4'] if use_initial_left_positions else 0.0}" />
-      <xacro:configure_rb_joint joint_name="left_manipulator_joint5" initial_value="${initial_positions['left_manipulator_joint5'] if use_initial_left_positions else 0.0}" />
-      <xacro:configure_rb_joint joint_name="left_manipulator_joint6" initial_value="${initial_positions['left_manipulator_joint6'] if use_initial_left_positions else 0.0}" />
+      <xacro:configure_rb_joint joint_name="left_manipulator_joint1" />
+      <xacro:configure_rb_joint joint_name="left_manipulator_joint2" />
+      <xacro:configure_rb_joint joint_name="left_manipulator_joint3" />
+      <xacro:configure_rb_joint joint_name="left_manipulator_joint4" />
+      <xacro:configure_rb_joint joint_name="left_manipulator_joint5" />
+      <xacro:configure_rb_joint joint_name="left_manipulator_joint6" />
     </ros2_control>
     <ros2_control name="RightRBPodoHardwareInterface" type="system">
@@ -56,10 +54,10 @@
         </xacro:unless>
       </hardware>
-      <xacro:configure_rb_joint joint_name="right_manipulator_joint1" initial_value="${initial_positions['right_manipulator_joint1'] if use_initial_right_positions else 0.0}" />
-      <xacro:configure_rb_joint joint_name="right_manipulator_joint2" initial_value="${initial_positions['right_manipulator_joint2'] if use_initial_right_positions else 0.0}" />
-      <xacro:configure_rb_joint joint_name="right_manipulator_joint3" initial_value="${initial_positions['right_manipulator_joint3'] if use_initial_right_positions else 0.0}" />
-      <xacro:configure_rb_joint joint_name="right_manipulator_joint4" initial_value="${initial_positions['right_manipulator_joint4'] if use_initial_right_positions else 0.0}" />
-      <xacro:configure_rb_joint joint_name="right_manipulator_joint5" initial_value="${initial_positions['right_manipulator_joint5'] if use_initial_right_positions else 0.0}" />
-      <xacro:configure_rb_joint joint_name="right_manipulator_joint6" initial_value="${initial_positions['right_manipulator_joint6'] if use_initial_right_positions else 0.0}" />
+      <xacro:configure_rb_joint joint_name="right_manipulator_joint1" />
+      <xacro:configure_rb_joint joint_name="right_manipulator_joint2" />
+      <xacro:configure_rb_joint joint_name="right_manipulator_joint3" />
+      <xacro:configure_rb_joint joint_name="right_manipulator_joint4" />
+      <xacro:configure_rb_joint joint_name="right_manipulator_joint5" />
+      <xacro:configure_rb_joint joint_name="right_manipulator_joint6" />
     </ros2_control>
     <!-- The two-axis head is MoveIt-only and never connects to an RB Control Box. -->

File: construct_moveit_config/config/construct_robot_0528.urdf.xacro (robot description, xacro)
@@ -4,10 +4,6 @@
     <xacro:arg name="left_robot_ip" default="192.168.1.11" />
     <xacro:arg name="cb_simulation" default="false" />
-    <xacro:arg name="use_fake_left_hardware" default="true" />
+    <xacro:arg name="use_fake_left_hardware" default="false" />
     <xacro:arg name="use_fake_right_hardware" default="false" />
-    <xacro:arg name="use_initial_left_positions" default="true" />
-    <xacro:arg name="use_initial_right_positions" default="true" />
-    <xacro:arg name="initial_positions_file"
-               default="$(find construct_description)/config/initial_positions.yaml" />
     <xacro:arg name="fake_sensor_commands" default="false" />
     <!-- Import construct_robot_0528 urdf file -->
@@ -21,7 +17,4 @@
         use_fake_left_hardware="$(arg use_fake_left_hardware)"
         use_fake_right_hardware="$(arg use_fake_right_hardware)"
-        use_initial_left_positions="$(arg use_initial_left_positions)"
-        use_initial_right_positions="$(arg use_initial_right_positions)"
-        initial_positions_file="$(arg initial_positions_file)"
         fake_sensor_commands="$(arg fake_sensor_commands)" />
 </robot>
