Commit message: linear welding motion

File: construct_description/urdf_0528/construct_robot_0528.urdf (robot description, URDF)
Before this commit: robot construct_robot_0528, 56 links, 55 joints
Links:
- link testbed_link: geometry collision mesh filename=package://construct_description/meshes_0528/testbed_link_op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
