Commit message: add head hardware

File: construct_description/urdf_0528/construct_robot_0528.ros2_control.xacro (robot description, xacro)
@@ -63,5 +63,5 @@
     <!-- The two-axis head is MoveIt-only and never connects to an RB Control Box. -->
     <ros2_control name="HeadMoveItSystem" type="system">
-      <hardware>
+      <!-- <hardware>
         <plugin>mock_components/GenericSystem</plugin>
         <param name="mock_sensor_commands">${fake_sensor_commands}</param>
@@ -81,5 +81,27 @@
           <param name="initial_value">0.0</param>
         </state_interface>
-      </joint>
+      </joint> -->
+        <hardware>
+            <plugin>kaiser_hardware/KaiserHardwareInterface</plugin>
+            <param name="can_interface">can2</param>
+        </hardware>
+        <joint name="robot_head_rev_joint1">
+            <param name="motor_id">2</param>
+            <command_interface name="position" />
+            <state_interface name="position" />
+            <state_interface name="velocity" />
+            <!-- <state_interface name="current" />
+            <state_interface name="status" />
+            <state_interface name="error" /> -->
+        </joint>
+        <joint name="robot_head_rev_joint2">
+            <param name="motor_id">1</param>
+            <command_interface name="position" />
+            <state_interface name="position" />
+            <state_interface name="velocity" />
+            <!-- <state_interface name="current" />
+            <state_interface name="status" />
+            <state_interface name="error" /> -->
+        </joint>
     </ros2_control>
   </xacro:macro>

File: construct_description/urdf_0528/construct_robot_0528.urdf (robot description, URDF)
Before this commit: robot construct_robot_0528, 56 links, 55 joints
Joints:
- joint robot_head_rev_joint2: axis 0 0 -1 -> 0 0 1

Commit message: add keyboard teleoperation

File: construct_description/urdf_0528/construct_robot_0528.ros2_control.xacro (robot description, xacro)
@@ -18,4 +18,17 @@
         </state_interface>
       </joint>
+    </xacro:macro>
+    <!-- The real RB adapter exports these six resources itself.  Declare the
+         same command resources for GenericSystem so fake-hardware tests can
+         exercise the exact trajectory <-> Cartesian-velocity switch. -->
+    <xacro:macro name="configure_fake_cartesian_velocity" params="arm enabled">
+      <xacro:if value="${enabled}">
+        <gpio name="${arm}/x"><command_interface name="cartesian_velocity" /></gpio>
+        <gpio name="${arm}/y"><command_interface name="cartesian_velocity" /></gpio>
+        <gpio name="${arm}/z"><command_interface name="cartesian_velocity" /></gpio>
+        <gpio name="${arm}/rx"><command_interface name="cartesian_velocity" /></gpio>
+        <gpio name="${arm}/ry"><command_interface name="cartesian_velocity" /></gpio>
+        <gpio name="${arm}/rz"><command_interface name="cartesian_velocity" /></gpio>
+      </xacro:if>
     </xacro:macro>
     <ros2_control name="LeftRBPodoHardwareInterface" type="system">
@@ -39,4 +52,5 @@
       <xacro:configure_rb_joint joint_name="left_manipulator_joint5" />
       <xacro:configure_rb_joint joint_name="left_manipulator_joint6" />
+      <xacro:configure_fake_cartesian_velocity arm="left" enabled="${use_fake_left_hardware}" />
     </ros2_control>
     <ros2_control name="RightRBPodoHardwareInterface" type="system">
@@ -60,4 +74,5 @@
       <xacro:configure_rb_joint joint_name="right_manipulator_joint5" />
       <xacro:configure_rb_joint joint_name="right_manipulator_joint6" />
+      <xacro:configure_fake_cartesian_velocity arm="right" enabled="${use_fake_right_hardware}" />
     </ros2_control>
     <!-- The two-axis head is MoveIt-only and never connects to an RB Control Box. -->
